Commit message: Test: add mimic expression.

File: fanuc_m900ib_support/urdf/m900ib700_macro.xacro (robot description, xacro)
@@ -273,5 +273,5 @@
       <child link="${prefix}balancer_left"/>
       <axis xyz="0 1 0"/>
-      <mimic joint="${prefix}joint_2" multiplier="0.18" offset="0" />
+      <mimic joint="${prefix}joint_2" multiplier="0.18" offset="0" expr="sin(${prefix}joint_1_q) + ${prefix}joint_3_q" />
     </joint>
     <joint name="${prefix}piston_left_joint" type="continuous">
